Commit message: Add D435 and remove T265

File: legged_perceptive_description/urdf/robot.xacro (robot description, xacro)
@@ -12,9 +12,12 @@
         <origin xyz="0.16 0 0.085" rpy="0 -1.04 0"/>
     </xacro:sensor_t265>
-    <xacro:mid360 name="livox_right" parent="base">
+    <!-- <xacro:mid360 name="livox_right" parent="base">
         <origin xyz="0.365 -0.068 -0.030" rpy="-2.59 1.03 3.09"/>
     </xacro:mid360>
     <xacro:mid360 name="livox_left" parent="base">
         <origin xyz="0.365 0.068 -0.030" rpy="2.59 1.03 -3.09"/>
-    </xacro:mid360>
+    </xacro:mid360> -->
+    <xacro:sensor_d435 name="rs_front" topics_ns="rs_front" parent="base">
+        <origin rpy="0.0 0.1 0.0" xyz="0.35 0 0.1"/>
+    </xacro:sensor_d435>
 </robot>

File: legged_perceptive_description/urdf/sensor_d435.xacro (robot description, xacro)
@@ -112,12 +112,17 @@
             </joint>
             <link name="${name}_color_optical_frame"/>
-            <xacro:include filename="$(find legged_perceptive_description)/urdf/gazebo_d400.xacro"/>
+            <xacro:include filename="$(find legged_perceptive_description)/urdf/gazebo_d435.xacro"/>
             <!-- Realsense Gazebo Plugin -->
-            <xacro:gazebo_d400 camera_name="${name}" reference_link="${name}_link" topics_ns="${topics_ns}"
+            <xacro:gazebo_d435 camera_name="${name}" reference_link="${name}_link" topics_ns="${topics_ns}"
+                               depth_optical_frame="${name}_depth_optical_frame"
+                               color_optical_frame="${name}_color_optical_frame"
+                               infrared1_optical_frame="${name}_left_ir_optical_frame"
+                               infrared2_optical_frame="${name}_right_ir_optical_frame"/>
+            <!-- <xacro:gazebo_d400 camera_name="${name}" reference_link="${name}_link" topics_ns="${topics_ns}"
                                depth_optical_frame="${name}_depth_optical_frame"
                                color_optical_frame="${name}_color_optical_frame"
                                infrared1_optical_frame="${name}_left_ir_optical_frame"
                                infrared2_optical_frame="${name}_right_ir_optical_frame"
-                               publish_pointcloud="${publish_pointcloud}"/>
+                               publish_pointcloud="${publish_pointcloud}"/> -->
         </xacro:if>
     </xacro:macro>

File: legged_perceptive_description/urdf/sensor_t265.xacro (robot description, xacro)
@@ -31,5 +31,5 @@
                 <origin xyz="0 0 0" rpy="0 0 0"/>
                 <geometry>
-                    <mesh filename="package://realsense2_description/meshes/t265.stl"/>
+                    <!-- <mesh filename="package://realsense2_description/meshes/t265.stl"/> -->
                 </geometry>
                 <material name="${name}_aluminum"/>
@@ -38,5 +38,5 @@
                 <origin xyz="0 0 0" rpy="0 0 0"/>
                 <geometry>
-                    <mesh filename="package://realsense2_description/meshes/t265.stl"/>
+                    <!-- <mesh filename="package://realsense2_description/meshes/t265.stl"/> -->
                 </geometry>
             </collision>
